Commit message: Set offset to M2 reference point

File: urdf/ev_nautilus_mesh.xacro (robot description, xacro)
@@ -6,6 +6,8 @@
     <visual>
         <geometry>
-            <mesh filename="package://ev_nautilus_description/models/meshes/nautilus.dae"/>
+            <mesh filename="package://ev_nautilus_description/models/meshes/nautilus.dae" scale="10 10 10"/>
         </geometry>
+        <!-- <origin rpy="0 0 -1.57075" xyz="-33.657 0.067 -2.628"/> -->
+        <origin rpy="0 0 -1.57075" xyz="-34.383 0.359 -0.013"/>
     </visual>
   </link>
